File: hw/USB2517.sch (KiCad schematic (older format))
At the start: 1 part

Commit message: Add more
Parts:
- removed U?: USB2517, symbol USB2517:USB2517
- added C1, C2, C7: 1uF, symbol Device:C_Small
- added C10, C9: 18pF, symbol Device:C_Small
- added C3, C4, C5, C6: 10uF, symbol Device:C_Small
- added C8: 0.1uF, symbol Device:C_Small
- added J1: Barrel_Jack, symbol Connector:Barrel_Jack
- added J2: USB_B_Micro, symbol Connector:USB_B_Micro
- added R0, R10, R9: 0R, symbol Device:R_Small
- added R1, R5, R7: 10k, symbol Device:R_Small
- added R11, R6, R8: DNP, symbol Device:R_Small
- added R2, R3: 100k, symbol Device:R_Small
- added R4: 12k 1%, symbol Device:R_Small
- added U1: MIC5219-3.3, Package_TO_SOT_SMD:SOT-23-5, symbol Regulator_Linear:MIC5219-3.3
- added U2: LM1085-5.0, symbol Regulator_Linear:LM1085-5.0
- added U3: USB2517, symbol USB2517:USB2517
- added U4: 24LC02, symbol Memory_EEPROM:24LC02
- added Y1: 24Mhz, symbol crystal_small_smd:Crystal_Small_SMD
Connections:
- net labels added: +3V3, +5V, EEPROM_SCL, EEPROM_SDA, GND, LOCAL_PWR, VBUS
- wire segments 0 -> 140
- no-connect marks 0 -> 2
Other:
- note added: "C_IN should be rated for at least 30v"
- note added: "Place either R0 or LM1085"
- note added: "Power for MCU and USB HUB"
- note added: "R0 must be able to handle 500mA at least"

Commit message: Finish up usb port hookup
Other:
- note added: "C5 should be rated for at least 30v"
- note removed: "C_IN should be rated for at least 30v"
Changed lines of the file:
@@
 Connection ~ 2300 1350
 Text Notes 600  950  0    50   ~ 0
-C_IN should be rated for at least 30v
+C5 should be rated for at least 30v
 $Comp
 L Device:R_Small R6

Commit message: minor fixes
Parts:
- added R12, R13: 10k, symbol Device:R_Small
Connections:
- wire segments 140 -> 146
Other:
- note added: "C5 should be rated for at least 16v"
- note removed: "C5 should be rated for at least 30v"
- moved on the sheet: R0
Changed lines of the file:
@@
 Text Label 3800 1700 0    50   ~ 0
 VBUS
-Text Label 750  2300 0    50   ~ 0
+Text Label 650  2250 0    50   ~ 0
 VBUS
 $Comp
 L Device:R_Small R0
 U 1 1 5B990046
-P 1100 2300
-F 0 "R0" V 1100 2300 50  0000 C CNN
-F 1 "0R" V 995 2300 50  0000 C CNN
-F 2 "" H 1100 2300 50  0001 C CNN
-F 3 "~" H 1100 2300 50  0001 C CNN
-	1    1100 2300
+P 1300 2250
+F 0 "R0" V 1300 2250 50  0000 C CNN
+F 1 "0R" V 1350 2100 50  0000 C CNN
+F 2 "" H 1300 2250 50  0001 C CNN
+F 3 "~" H 1300 2250 50  0001 C CNN
+	1    1300 2250
 	0    1    1    0
 $EndComp
@@
 L power:+5V #PWR010
 U 1 1 5B990107
-P 1450 2200
-F 0 "#PWR010" H 1450 2050 50  0001 C CNN
-F 1 "+5V" H 1465 2373 50  0000 C CNN
-F 2 "" H 1450 2200 50  0001 C CNN
-F 3 "" H 1450 2200 50  0001 C CNN
-	1    1450 2200
-	1    0    0    -1
-$EndComp
-Wire Wire Line
-	750  2300 1000 2300
-Wire Wire Line
-	1200 2300 1450 2300
-Wire Wire Line
-	1450 2300 1450 2200
+P 1550 2250
+F 0 "#PWR010" H 1550 2100 50  0001 C CNN
+F 1 "+5V" H 1565 2423 50  0000 C CNN
+F 2 "" H 1550 2250 50  0001 C CNN
+F 3 "" H 1550 2250 50  0001 C CNN
+	1    1550 2250
+	0    1    1    0
+$EndComp
+Wire Wire Line
+	650  2250 1200 2250
+Wire Wire Line
+	1400 2250 1550 2250
 Wire Notes Line
 	2500 2500 550  2500
-Wire Notes Line
-	550  2500 550  750
 Wire Notes Line
 	550  750  2500 750
@@
 Wire Notes Line
 	2650 3850 550  3850
-Wire Notes Line
-	550  3850 550  2600
 $Comp
 L Device:C_Small C6
@@
 	1    0    0    -1
 $EndComp
-Wire Wire Line
-	1350 1750 1500 1750
 $Comp
 L Device:C_Small C5
@@
 Wire Wire Line
 	1500 1650 1500 1750
-Connection ~ 1500 1750
 Wire Wire Line
 	1500 1750 1900 1750
@@
 Connection ~ 2300 1350
 Text Notes 600  950  0    50   ~ 0
-C5 should be rated for at least 30v
+C5 should be rated for at least 16v
 $Comp
 L Device:R_Small R6
@@
 	4550 2550 4400 2550
 Connection ~ 4550 2550
+Text Label 650  1900 0    50   ~ 0
+LOCAL_PWR
+$Comp
+L Device:R_Small R12
+U 1 1 5BABDBC0
+P 1300 1900
+F 0 "R12" V 1300 1900 50  0000 C CNN
+F 1 "10k" V 1350 1750 50  0000 C CNN
+F 2 "" H 1300 1900 50  0001 C CNN
+F 3 "~" H 1300 1900 50  0001 C CNN
+	1    1300 1900
+	0    1    1    0
+$EndComp
+$Comp
+L power:+5V #PWR049
+U 1 1 5BAC2D8D
+P 1550 1900
+F 0 "#PWR049" H 1550 1750 50  0001 C CNN
+F 1 "+5V" H 1565 2073 50  0000 C CNN
+F 2 "" H 1550 1900 50  0001 C CNN
+F 3 "" H 1550 1900 50  0001 C CNN
+	1    1550 1900
+	0    1    1    0
+$EndComp
+Wire Wire Line
+	1200 1900 1000 1900
+Wire Wire Line
+	1400 1900 1550 1900
+Wire Notes Line
+	550  900  550  3850
+$Comp
+L Device:R_Small R13
+U 1 1 5BADCB28
+P 1300 2050
+F 0 "R13" V 1300 2050 50  0000 C CNN
+F 1 "10k" V 1350 1900 50  0000 C CNN
+F 2 "" H 1300 2050 50  0001 C CNN
+F 3 "~" H 1300 2050 50  0001 C CNN
+	1    1300 2050
+	0    1    1    0
+$EndComp
+$Comp
+L power:GND #PWR050
+U 1 1 5BADCBF7
+P 1550 2050
+F 0 "#PWR050" H 1550 1800 50  0001 C CNN
+F 1 "GND" V 1555 1922 50  0000 R CNN
+F 2 "" H 1550 2050 50  0001 C CNN
+F 3 "" H 1550 2050 50  0001 C CNN
+	1    1550 2050
+	0    -1   -1   0
+$EndComp
+Wire Wire Line
+	1550 2050 1400 2050
+Wire Wire Line
+	1200 2050 1000 2050
+Wire Wire Line
+	1000 2050 1000 1900
+Connection ~ 1000 1900
+Wire Wire Line
+	1000 1900 650  1900
+Wire Wire Line
+	1350 1750 1500 1750
+Connection ~ 1500 1750
+$Comp
+L power:PWR_FLAG #FLG0101
+U 1 1 5BAFE3BA
+P 1500 1250
+F 0 "#FLG0101" H 1500 1325 50  0001 C CNN
+F 1 "PWR_FLAG" H 1500 1424 50  0000 C CNN
+F 2 "" H 1500 1250 50  0001 C CNN
+F 3 "~" H 1500 1250 50  0001 C CNN
+	1    1500 1250
+	1    0    0    -1
+$EndComp
+Wire Wire Line
+	1500 1250 1500 1350
 $EndSCHEMATC

Commit message: Finalize schematics
Parts:
- added D7: PWR_LED_5V, symbol Device:LED_Small
- added D8: PWR_LED_3v, symbol Device:LED_Small
- added R19: 2.2k, symbol Device:R_Small
- added R20: 360R, symbol Device:R_Small
Connections:
- wire segments 146 -> 156
Changed lines of the file:
@@
 Wire Wire Line
 	1500 1250 1500 1350
+$Comp
+L Device:R_Small R19
+U 1 1 5BDCCDF2
+P 1100 4550
+F 0 "R19" V 904 4550 50  0000 C CNN
+F 1 "2.2k" V 995 4550 50  0000 C CNN
+F 2 "" H 1100 4550 50  0001 C CNN
+F 3 "~" H 1100 4550 50  0001 C CNN
+	1    1100 4550
+	0    1    1    0
+$EndComp
+$Comp
+L Device:LED_Small D7
+U 1 1 5BDCD10A
+P 1550 4550
+F 0 "D7" H 1550 4345 50  0000 C CNN
+F 1 "PWR_LED_5V" H 1550 4436 50  0000 C CNN
+F 2 "" V 1550 4550 50  0001 C CNN
+F 3 "~" V 1550 4550 50  0001 C CNN
+	1    1550 4550
+	-1   0    0    1
+$EndComp
+$Comp
+L power:GND #PWR0102
+U 1 1 5BDCD220
+P 1750 4700
+F 0 "#PWR0102" H 1750 4450 50  0001 C CNN
+F 1 "GND" H 1755 4527 50  0000 C CNN
+F 2 "" H 1750 4700 50  0001 C CNN
+F 3 "" H 1750 4700 50  0001 C CNN
+	1    1750 4700
+	1    0    0    -1
+$EndComp
+Wire Wire Line
+	1650 4550 1750 4550
+Wire Wire Line
+	1750 4550 1750 4700
+Wire Wire Line
+	1450 4550 1200 4550
+$Comp
+L power:+5V #PWR0103
+U 1 1 5BDD9085
+P 850 4450
+F 0 "#PWR0103" H 850 4300 50  0001 C CNN
+F 1 "+5V" H 865 4623 50  0000 C CNN
+F 2 "" H 850 4450 50  0001 C CNN
+F 3 "" H 850 4450 50  0001 C CNN
+	1    850  4450
+	1    0    0    -1
+$EndComp
+Wire Wire Line
+	850  4450 850  4550
+Wire Wire Line
+	850  4550 1000 4550
+$Comp
+L Device:R_Small R20
+U 1 1 5BDDF895
+P 1100 5250
+F 0 "R20" V 904 5250 50  0000 C CNN
+F 1 "360R" V 995 5250 50  0000 C CNN
+F 2 "" H 1100 5250 50  0001 C CNN
+F 3 "~" H 1100 5250 50  0001 C CNN
+	1    1100 5250
+	0    1    1    0
+$EndComp
+$Comp
+L Device:LED_Small D8
+U 1 1 5BDDF89B
+P 1550 5250
+F 0 "D8" H 1550 5045 50  0000 C CNN
+F 1 "PWR_LED_3v" H 1550 5136 50  0000 C CNN
+F 2 "" V 1550 5250 50  0001 C CNN
+F 3 "~" V 1550 5250 50  0001 C CNN
+	1    1550 5250
+	-1   0    0    1
+$EndComp
+$Comp
+L power:GND #PWR0104
+U 1 1 5BDDF8A1
+P 1750 5400
+F 0 "#PWR0104" H 1750 5150 50  0001 C CNN
+F 1 "GND" H 1755 5227 50  0000 C CNN
+F 2 "" H 1750 5400 50  0001 C CNN
+F 3 "" H 1750 5400 50  0001 C CNN
+	1    1750 5400
+	1    0    0    -1
+$EndComp
+Wire Wire Line
+	1650 5250 1750 5250
+Wire Wire Line
+	1750 5250 1750 5400
+Wire Wire Line
+	1450 5250 1200 5250
+Wire Wire Line
+	850  5250 1000 5250
+$Comp
+L power:+3V3 #PWR0105
+U 1 1 5BDE64BD
+P 850 5050
+F 0 "#PWR0105" H 850 4900 50  0001 C CNN
+F 1 "+3V3" H 865 5223 50  0000 C CNN
+F 2 "" H 850 5050 50  0001 C CNN
+F 3 "" H 850 5050 50  0001 C CNN
+	1    850  5050
+	1    0    0    -1
+$EndComp
+Wire Wire Line
+	850  5050 850  5250
 $EndSCHEMATC

Commit message: Add most footprints, switch to usb c
Parts:
- removed J2: USB_B_Micro, symbol Connector:USB_B_Micro
- added C21: 10uF, Capacitor_SMD:C_0603_1608Metric, symbol Device:C_Small
- added C22, C23, C24, C25, C26, C27, C28: 0.1uF, Capacitor_SMD:C_0603_1608Metric, symbol Device:C_Small
- added J2: USB_C_Receptacle, symbol Connector:USB_C_Receptacle
- added R29, R30: 5.11k, symbol Device:R_Small
- C1, C10, C2, C3, C4, C5, C6, C7, C8, C9: footprint (none) -> Capacitor_SMD:C_0603_1608Metric
- D7, D8: footprint (none) -> LED_SMD:LED_0603_1608Metric
- R0, R1, R10, R11, R12, R13, R19, R2, R20, R3, R4, R5, R6, R7, R8, R9: footprint (none) -> Resistor_SMD:R_0603_1608Metric
- U2: footprint (none) -> Package_TO_SOT_SMD:TO-263-3_TabPin2
- U3: footprint (none) -> Package_DFN_QFN:QFN-64-1EP_9x9mm_P0.5mm_EP4.7x4.7mm_ThermalVias
- U4: footprint (none) -> Package_SO:SOIC-8_3.9x4.9mm_P1.27mm
Connections:
- wire segments 156 -> 206
- no-connect marks 2 -> 11
Other:
- moved on the sheet: C1, C10, C2, C3, C4, C5, C6, C7, C8, C9, D7, D8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

Commit message: Add footprints to everything else, except barrel jack
Parts:
- J2: footprint (none) -> USB_C:USB_C_Receptacle_GT-USB-7010
- R29, R30: footprint (none) -> Resistor_SMD:R_0603_1608Metric
- Y1: footprint (none) -> Crystal:Crystal_SMD_2016-4Pin_2.0x1.6mm
Changed lines of the file:
@@
 F 0 "Y1" V 7404 4087 50  0000 L CNN
 F 1 "24Mhz" V 7495 4087 50  0000 L CNN
-F 2 "" H 7450 4000 50  0001 C CNN
+F 2 "Crystal:Crystal_SMD_2016-4Pin_2.0x1.6mm" H 7450 4000 50  0001 C CNN
 F 3 "" H 7450 4000 50  0000 C CNN
 	1    7450 4000
@@
 F 0 "J2" H 5805 5467 50  0000 C CNN
 F 1 "USB_C_Receptacle" H 5805 5376 50  0000 C CNN
-F 2 "" H 5850 3900 50  0001 C CNN
+F 2 "USB_C:USB_C_Receptacle_GT-USB-7010" H 5850 3900 50  0001 C CNN
 F 3 "http://www.usb.org/developers/docs/usb_31_033017.zip" H 5850 3900 50  0001 C CNN
 	1    5700 3900
@@
 F 0 "R29" V 6450 3100 50  0000 C CNN
 F 1 "5.11k" V 6345 3100 50  0000 C CNN
-F 2 "" H 6450 3100 50  0001 C CNN
+F 2 "Resistor_SMD:R_0603_1608Metric" H 6450 3100 50  0001 C CNN
 F 3 "~" H 6450 3100 50  0001 C CNN
 	1    6450 3100
@@
 F 0 "R30" V 6450 3200 50  0000 C CNN
 F 1 "5.11k" V 6550 3200 50  0000 C CNN
-F 2 "" H 6450 3200 50  0001 C CNN
+F 2 "Resistor_SMD:R_0603_1608Metric" H 6450 3200 50  0001 C CNN
 F 3 "~" H 6450 3200 50  0001 C CNN
 	1    6450 3200

Commit message: Add 3d models
Parts:
- removed J1: Barrel_Jack, symbol Connector:Barrel_Jack
- removed J2: USB_C_Receptacle, USB_C:USB_C_Receptacle_GT-USB-7010, symbol Connector:USB_C_Receptacle
- added J1: EXT_PWR, Connector_BarrelJack_Extra:Boom_Precision_Elec_DC-005_5.5-2.0MM, symbol Connector:Barrel_Jack_Switch
- added J2: USB_C_Receptacle_USB2.0, USB_C:USB_C_Receptacle_GT-USB-7010, symbol Connector:USB_C_Receptacle_USB2.0
- U1: symbol Regulator_Linear:MIC5219-3.3 -> Regulator_Linear:MIC5219-3.3YM5
Connections:
- wire segments 206 -> 194
- no-connect marks 11 -> 4
Other:
- note added: "Power for USB HUB"
- note removed: "Power for MCU and USB HUB"
Changed lines of the file:
@@
 	7350 3000 7300 3000
 $Comp
-L Regulator_Linear:MIC5219-3.3 U1
+L Regulator_Linear:MIC5219-3.3YM5 U1
 U 1 1 5B95DE23
 P 2000 4600
+AR Path="/5B95DE23" Ref="U1"  Part="1"
+AR Path="/5A7CEC76/5B95DE23" Ref="U1"  Part="1"
 F 0 "U1" H 2000 4942 50  0000 C CNN
 F 1 "MIC5219-3.3" H 2000 4851 50  0000 C CNN
@@
 Wire Wire Line
 	1150 5000 2000 5000
-$Comp
-L Connector:Barrel_Jack J1
-U 1 1 5B980A1C
-P 1300 2950
-F 0 "J1" H 1355 3275 50  0000 C CNN
-F 1 "Barrel_Jack" H 1355 3184 50  0000 C CNN
-F 2 "" H 1350 2910 50  0001 C CNN
-F 3 "~" H 1350 2910 50  0001 C CNN
-	1    1300 2950
-	1    0    0    -1
-$EndComp
-Wire Wire Line
-	1600 2850 1750 2850
 $Comp
 L power:GND #PWR08
@@
 Connection ~ 8800 4900
 Text Notes 1000 4200 0    50   ~ 0
-Power for MCU and USB HUB
+Power for USB HUB
 Wire Notes Line
 	800  4100 2900 4100
@@
 Wire Wire Line
 	1550 1250 1150 1250
-$Comp
-L Connector:USB_C_Receptacle J2
-U 1 1 5BE19532
-P 5700 3900
-F 0 "J2" H 5805 5467 50  0000 C CNN
-F 1 "USB_C_Receptacle" H 5805 5376 50  0000 C CNN
-F 2 "USB_C:USB_C_Receptacle_GT-USB-7010" H 5850 3900 50  0001 C CNN
-F 3 "http://www.usb.org/developers/docs/usb_31_033017.zip" H 5850 3900 50  0001 C CNN
-	1    5700 3900
-	1    0    0    -1
-$EndComp
-NoConn ~ 6300 3900
-NoConn ~ 6300 4000
-NoConn ~ 6300 4200
-NoConn ~ 6300 4300
-NoConn ~ 6300 4500
-NoConn ~ 6300 4600
-NoConn ~ 6300 4800
-NoConn ~ 6300 4900
-NoConn ~ 6300 5100
-NoConn ~ 6300 5200
-$Comp
-L power:GND #PWR064
-U 1 1 5BE966B3
-P 5800 5950
-F 0 "#PWR064" H 5800 5700 50  0001 C CNN
-F 1 "GND" H 5805 5777 50  0000 C CNN
-F 2 "" H 5800 5950 50  0001 C CNN
-F 3 "" H 5800 5950 50  0001 C CNN
-	1    5800 5950
-	1    0    0    -1
-$EndComp
-Wire Wire Line
-	5800 5500 5800 5700
-Wire Wire Line
-	5400 5500 5400 5700
-Wire Wire Line
-	5400 5700 5500 5700
-Connection ~ 5800 5700
-Wire Wire Line
-	5800 5700 5800 5950
-Wire Wire Line
-	5500 5500 5500 5700
-Connection ~ 5500 5700
-Wire Wire Line
-	5500 5700 5600 5700
-Wire Wire Line
-	5600 5500 5600 5700
-Connection ~ 5600 5700
-Wire Wire Line
-	5600 5700 5700 5700
-Wire Wire Line
-	5700 5550 5700 5700
-Connection ~ 5700 5700
-Wire Wire Line
-	5700 5700 5800 5700
 Wire Wire Line
 	6300 3500 6450 3500
@@
 Wire Wire Line
 	7050 3000 7050 2900
-Wire Wire Line
-	7050 2900 6450 2900
 Connection ~ 7050 3000
-Wire Wire Line
-	6450 2900 6450 2800
-Wire Wire Line
-	6450 2600 6300 2600
-Connection ~ 6450 2900
-Wire Wire Line
-	6450 2900 6300 2900
-Wire Wire Line
-	6300 2700 6450 2700
-Connection ~ 6450 2700
-Wire Wire Line
-	6450 2700 6450 2600
-Wire Wire Line
-	6300 2800 6450 2800
-Connection ~ 6450 2800
-Wire Wire Line
-	6450 2800 6450 2700
 Wire Wire Line
 	6300 3400 6450 3400
@@
 Wire Wire Line
 	6700 3200 6700 3300
+$Comp
+L Connector:Barrel_Jack_Switch J1
+U 1 1 5BD9F088
+P 1150 2950
+F 0 "J1" H 1205 3267 50  0000 C CNN
+F 1 "EXT_PWR" H 1205 3176 50  0000 C CNN
+F 2 "Connector_BarrelJack_Extra:Boom_Precision_Elec_DC-005_5.5-2.0MM" H 1200 2910 50  0001 C CNN
+F 3 "~" H 1200 2910 50  0001 C CNN
+	1    1150 2950
+	1    0    0    -1
+$EndComp
+$Comp
+L Connector:USB_C_Receptacle_USB2.0 J2
+U 1 1 5BDA05D7
+P 5700 3500
+F 0 "J2" H 5805 4367 50  0000 C CNN
+F 1 "USB_C_Receptacle_USB2.0" H 5805 4276 50  0000 C CNN
+F 2 "USB_C:USB_C_Receptacle_GT-USB-7010" H 5850 3500 50  0001 C CNN
+F 3 "https://www.usb.org/sites/default/files/documents/usb_type-c.zip" H 5850 3500 50  0001 C CNN
+	1    5700 3500
+	1    0    0    -1
+$EndComp
+Wire Wire Line
+	6300 2900 7050 2900
+NoConn ~ 6300 4000
+NoConn ~ 6300 4100
+$Comp
+L power:GND #PWR064
+U 1 1 5BDE08D3
+P 5700 4650
+F 0 "#PWR064" H 5700 4400 50  0001 C CNN
+F 1 "GND" H 5705 4477 50  0000 C CNN
+F 2 "" H 5700 4650 50  0001 C CNN
+F 3 "" H 5700 4650 50  0001 C CNN
+	1    5700 4650
+	1    0    0    -1
+$EndComp
+Wire Wire Line
+	5700 4400 5700 4550
+Wire Wire Line
+	5700 4550 5400 4550
+Wire Wire Line
+	5400 4550 5400 4400
+Connection ~ 5700 4550
+Wire Wire Line
+	5700 4550 5700 4650
+Wire Wire Line
+	1450 2850 1750 2850
+Wire Wire Line
+	1600 3050 1450 3050
+NoConn ~ 1450 2950
 $EndSCHEMATC

Commit message: Begin routing
Connections:
- net EXT_PWR: now reaches C5.1, J1.1, U2.3 (VI)
Changed lines of the file:
@@
 	1600 3050 1450 3050
 NoConn ~ 1450 2950
+Text Label 1550 2850 1    50   ~ 0
+EXT_PWR
 $EndSCHEMATC
