File: hw/_autosave-usbhub.kicad_pcb (KiCad board)
At the start: 2 copper layers, 100 x 100 mm, 92 parts, among them J1 EXT_PWR, J2 USB_C_Receptacle_USB2.0, J3 USB6, J4 USB2, J5 USB7, J6 USB3, J7 USB4, J8 USB5, J9 SWD, SW1 SW_Push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

Commit message: Begin routing
Parts:
- moved U11 69.9 mm to (161.4, 105.9), turned to 270 degrees
- moved J4 60.0 mm to (190.0, 123.0)
- moved J8 60.0 mm to (190.0, 63.0)
- moved U10 60.0 mm to (183.0, 63.0)
- moved U5 60.0 mm to (183.0, 123.0)
- moved U6 40.0 mm to (177.0, 113.0)
- moved U9 40.0 mm to (177.0, 73.0)
- moved J6 20.0 mm to (190.0, 103.0)
- moved J7 20.0 mm to (190.0, 83.0)
- moved U7 20.0 mm to (183.0, 103.0)
- moved U8 20.0 mm to (183.0, 83.0)
Connections:
- U6 pad 5: /USBPorts/USB3_VBUS -> /USBPorts/USB2_VBUS
- U6 pad 8: /USBPorts/USB2_VBUS -> /USBPorts/USB3_VBUS
- U9 pad 5: /USBPorts/USB5_VBUS -> /USBPorts/USB4_VBUS
- U9 pad 8: /USBPorts/USB4_VBUS -> /USBPorts/USB5_VBUS
