File: hw/MCU.sch (KiCad schematic (older format))
At the start: 1 part, among them U11 EFM32HG310F64G-B-QFN32

Commit message: minor fixes
Parts:
- added C?: C_Small, symbol Device:C_Small
- added R? (x2): 27R, symbol Device:R_Small
- added U?: USB2517, symbol USB2517:USB2517
Connections:
- net labels added: GND, MCU_SWDCLK, MCU_SWDIO, PORT2_EN, PORT2_PWR, USB_MCU_D+, USB_MCU_D-, VBUSDETECT
- wire segments 0 -> 20
- no-connect marks 0 -> 3
Changed lines of the file:
@@
 	1    0    0    -1
 $EndComp
+$Comp
+L power:GND #PWR?
+U 1 1 5BB092EA
+P 4650 5050
+F 0 "#PWR?" H 4650 4800 50  0001 C CNN
+F 1 "GND" H 4655 4877 50  0000 C CNN
+F 2 "" H 4650 5050 50  0001 C CNN
+F 3 "" H 4650 5050 50  0001 C CNN
+	1    4650 5050
+	1    0    0    -1
+$EndComp
+Wire Wire Line
+	4550 4400 4550 4950
+Wire Wire Line
+	4550 4950 4650 4950
+Wire Wire Line
+	4650 4950 4650 5050
+$Comp
+L USB2517:USB2517 U?
+U 2 1 5BB8A495
+P 7150 3650
+F 0 "U?" H 6823 3604 50  0000 R CNN
+F 1 "USB2517" H 6823 3695 50  0000 R CNN
+F 2 "" H 8250 5450 50  0001 C CNN
+F 3 "" H 8250 5450 50  0001 C CNN
+	2    7150 3650
+	-1   0    0    1
+$EndComp
+Text Label 5600 3400 0    50   ~ 0
+USB_MCU_D+
+Text Label 5600 3500 0    50   ~ 0
+USB_MCU_D-
+NoConn ~ 6700 3700
+NoConn ~ 6700 3800
+NoConn ~ 6700 3900
+Wire Wire Line
+	5450 3000 6200 3000
+Wire Wire Line
+	5450 3100 6200 3100
+Text Label 5550 3000 0    50   ~ 0
+MCU_SWDIO
+Text Label 5550 3100 0    50   ~ 0
+MCU_SWDCLK
+Wire Wire Line
+	6700 3600 5450 3600
+Text Label 5600 3600 0    50   ~ 0
+VBUSDETECT
+Text HLabel 3350 2500 0    50   Input ~ 0
+PORT2_PWR
+Text HLabel 3350 2600 0    50   Input ~ 0
+PORT2_PWR
+Text HLabel 3350 2700 0    50   Input ~ 0
+PORT2_PWR
+Text HLabel 3350 2800 0    50   Input ~ 0
+PORT2_PWR
+Text HLabel 3350 3500 0    50   Input ~ 0
+PORT2_EN
+Text HLabel 3350 3600 0    50   Input ~ 0
+PORT2_EN
+Text HLabel 3350 3700 0    50   Input ~ 0
+PORT2_EN
+Text HLabel 3350 3800 0    50   Input ~ 0
+PORT2_EN
+Wire Wire Line
+	3800 3500 3350 3500
+Wire Wire Line
+	3350 3600 3800 3600
+Wire Wire Line
+	3800 3700 3350 3700
+Wire Wire Line
+	3800 3800 3350 3800
+Wire Wire Line
+	3350 2500 3800 2500
+Wire Wire Line
+	3350 2600 3800 2600
+Wire Wire Line
+	3350 2700 3800 2700
+Wire Wire Line
+	3800 2800 3350 2800
+$Comp
+L Device:C_Small C?
+U 1 1 5BC29C29
+P 4650 4600
+F 0 "C?" H 4742 4646 50  0000 L CNN
+F 1 "C_Small" H 4742 4555 50  0000 L CNN
+F 2 "" H 4650 4600 50  0001 C CNN
+F 3 "~" H 4650 4600 50  0001 C CNN
+	1    4650 4600
+	1    0    0    -1
+$EndComp
+Wire Wire Line
+	4650 4400 4650 4500
+Wire Wire Line
+	4650 4700 4650 4950
+Connection ~ 4650 4950
+$Comp
+L Device:R_Small R?
+U 1 1 5BC2A861
+P 6350 3400
+F 0 "R?" V 6154 3400 50  0000 C CNN
+F 1 "27R" V 6245 3400 50  0000 C CNN
+F 2 "" H 6350 3400 50  0001 C CNN
+F 3 "~" H 6350 3400 50  0001 C CNN
+	1    6350 3400
+	0    1    1    0
+$EndComp
+$Comp
+L Device:R_Small R?
+U 1 1 5BC2A890
+P 6350 3500
+F 0 "R?" V 6500 3500 50  0000 C CNN
+F 1 "27R" V 6600 3500 50  0000 C CNN
+F 2 "" H 6350 3500 50  0001 C CNN
+F 3 "~" H 6350 3500 50  0001 C CNN
+	1    6350 3500
+	0    1    1    0
+$EndComp
+Wire Wire Line
+	6700 3400 6450 3400
+Wire Wire Line
+	6700 3500 6450 3500
+Wire Wire Line
+	6250 3500 5450 3500
+Wire Wire Line
+	6250 3400 5450 3400
 $EndSCHEMATC

Commit message: Finalize schematics
Parts:
- removed R? (x2): 27R, symbol Device:R_Small
- added C16: 10uF, symbol Device:C_Small
- added C17, C18, C20: 0.1uF, symbol Device:C_Small
- added C19: 4.7uF, symbol Device:C_Small
- added D2: Green, symbol Device:LED_Small
- added D3, D4, D5, D6: LED_Small, symbol Device:LED_Small
- added J9: SWD, symbol Connector_Generic:Conn_01x04
- added R14, R15: 360R, symbol Device:R_Small
- added R16, R17, R18: R_Small, symbol Device:R_Small
- added SW1: SW_Push, symbol Switch:SW_Push
- gave numbers to parts that had none: 2
Connections:
- net labels added: +5V, DECOUPLE, PORT3_EN, PORT3_PWR, PORT4_EN, PORT4_PWR, PORT5_EN, PORT5_PWR, VDDMCU
- wire segments 20 -> 93
- no-connect marks 3 -> 12

Commit message: Add most footprints, switch to usb c
Parts:
- C15, C16, C17, C18, C19, C20: footprint (none) -> Capacitor_SMD:C_0603_1608Metric
- D2, D3, D4, D5, D6: footprint (none) -> LED_SMD:LED_0603_1608Metric
- J9: footprint (none) -> Connector_JST:JST_SH_BM04B-SRSS-TB_1x04-1MP_P1.00mm_Vertical
- R14, R15, R16, R17, R18: footprint (none) -> Resistor_SMD:R_0603_1608Metric
- SW1: footprint (none) -> Button_Switch_SMD:SW_SPST_B3U-1000P
- U11: footprint (none) -> Package_DFN_QFN_Extra:QFN-32_EP_6x6_Pitch0.65mm
- U3: footprint (none) -> Package_DFN_QFN:QFN-64-1EP_9x9mm_P0.5mm_EP4.7x4.7mm_ThermalVias
Changed lines of the file:
@@
 F 0 "U11" H 5200 2250 50  0000 C CNN
 F 1 "EFM32HG310F64G-B-QFN32" V 4450 3200 50  0000 C CNN
-F 2 "" H 4550 3250 50  0001 C CNN
+F 2 "Package_DFN_QFN_Extra:QFN-32_EP_6x6_Pitch0.65mm" H 4550 3250 50  0001 C CNN
 F 3 "" H 4550 3250 50  0001 C CNN
 	1    4600 3250
@@
 F 0 "U3" H 6823 3604 50  0000 R CNN
 F 1 "USB2517" H 6823 3695 50  0000 R CNN
-F 2 "" H 8250 5450 50  0001 C CNN
+F 2 "Package_DFN_QFN:QFN-64-1EP_9x9mm_P0.5mm_EP4.7x4.7mm_ThermalVias" H 8250 5450 50  0001 C CNN
 F 3 "" H 8250 5450 50  0001 C CNN
 	2    7150 3650
@@
 F 0 "C15" H 4742 4646 50  0000 L CNN
 F 1 "C_Small" H 4742 4555 50  0000 L CNN
-F 2 "" H 4650 4600 50  0001 C CNN
+F 2 "Capacitor_SMD:C_0603_1608Metric" H 4650 4600 50  0001 C CNN
 F 3 "~" H 4650 4600 50  0001 C CNN
 	1    4650 4600
@@
 F 0 "J9" H 6780 1892 50  0000 L CNN
 F 1 "SWD" H 6780 1801 50  0000 L CNN
-F 2 "" H 6700 1900 50  0001 C CNN
+F 2 "Connector_JST:JST_SH_BM04B-SRSS-TB_1x04-1MP_P1.00mm_Vertical" H 6700 1900 50  0001 C CNN
 F 3 "~" H 6700 1900 50  0001 C CNN
 	1    6700 1900
@@
 F 0 "R14" V 5650 2250 50  0000 C CNN
 F 1 "360R" V 5700 2250 50  0000 C CNN
-F 2 "" H 5650 2250 50  0001 C CNN
+F 2 "Resistor_SMD:R_0603_1608Metric" H 5650 2250 50  0001 C CNN
 F 3 "~" H 5650 2250 50  0001 C CNN
 	1    5650 2250
@@
 F 0 "D2" H 6100 2300 50  0000 C CNN
 F 1 "Green" H 6000 2400 50  0000 C CNN
-F 2 "" V 6000 2250 50  0001 C CNN
+F 2 "LED_SMD:LED_0603_1608Metric" V 6000 2250 50  0001 C CNN
 F 3 "~" V 6000 2250 50  0001 C CNN
 	1    6000 2250
@@
 F 0 "C16" H 1042 1046 50  0000 L CNN
 F 1 "10uF" H 1042 955 50  0000 L CNN
-F 2 "" H 950 1000 50  0001 C CNN
+F 2 "Capacitor_SMD:C_0603_1608Metric" H 950 1000 50  0001 C CNN
 F 3 "~" H 950 1000 50  0001 C CNN
 	1    950  1000
@@
 F 0 "C17" H 1342 1046 50  0000 L CNN
 F 1 "0.1uF" H 1342 955 50  0000 L CNN
-F 2 "" H 1250 1000 50  0001 C CNN
+F 2 "Capacitor_SMD:C_0603_1608Metric" H 1250 1000 50  0001 C CNN
 F 3 "~" H 1250 1000 50  0001 C CNN
 	1    1250 1000
@@
 F 0 "C18" H 1642 1046 50  0000 L CNN
 F 1 "0.1uF" H 1642 955 50  0000 L CNN
-F 2 "" H 1550 1000 50  0001 C CNN
+F 2 "Capacitor_SMD:C_0603_1608Metric" H 1550 1000 50  0001 C CNN
 F 3 "~" H 1550 1000 50  0001 C CNN
 	1    1550 1000
@@
 F 0 "C19" H 1892 1046 50  0000 L CNN
 F 1 "4.7uF" H 1892 955 50  0000 L CNN
-F 2 "" H 1800 1000 50  0001 C CNN
+F 2 "Capacitor_SMD:C_0603_1608Metric" H 1800 1000 50  0001 C CNN
 F 3 "~" H 1800 1000 50  0001 C CNN
 	1    1800 1000
@@
 F 0 "C20" H 2192 1046 50  0000 L CNN
 F 1 "0.1uF" H 2192 955 50  0000 L CNN
-F 2 "" H 2100 1000 50  0001 C CNN
+F 2 "Capacitor_SMD:C_0603_1608Metric" H 2100 1000 50  0001 C CNN
 F 3 "~" H 2100 1000 50  0001 C CNN
 	1    2100 1000
@@
 F 0 "R15" V 3350 2500 50  0000 C CNN
 F 1 "360R" V 3245 2500 50  0000 C CNN
-F 2 "" H 3350 2500 50  0001 C CNN
+F 2 "Resistor_SMD:R_0603_1608Metric" H 3350 2500 50  0001 C CNN
 F 3 "~" H 3350 2500 50  0001 C CNN
 	1    3350 2500
@@
 F 0 "R16" V 3154 2700 50  0000 C CNN
 F 1 "R_Small" V 3245 2700 50  0000 C CNN
-F 2 "" H 3350 2700 50  0001 C CNN
+F 2 "Resistor_SMD:R_0603_1608Metric" H 3350 2700 50  0001 C CNN
 F 3 "~" H 3350 2700 50  0001 C CNN
 	1    3350 2700
@@
 F 0 "R17" V 3154 2800 50  0000 C CNN
 F 1 "R_Small" V 3245 2800 50  0000 C CNN
-F 2 "" H 3350 2800 50  0001 C CNN
+F 2 "Resistor_SMD:R_0603_1608Metric" H 3350 2800 50  0001 C CNN
 F 3 "~" H 3350 2800 50  0001 C CNN
 	1    3350 2800
@@
 F 0 "R18" V 3154 3000 50  0000 C CNN
 F 1 "R_Small" V 3245 3000 50  0000 C CNN
-F 2 "" H 3350 3000 50  0001 C CNN
+F 2 "Resistor_SMD:R_0603_1608Metric" H 3350 3000 50  0001 C CNN
 F 3 "~" H 3350 3000 50  0001 C CNN
 	1    3350 3000
@@
 F 0 "D6" H 2650 3235 50  0000 C CNN
 F 1 "LED_Small" H 2650 3144 50  0000 C CNN
-F 2 "" V 2650 3000 50  0001 C CNN
+F 2 "LED_SMD:LED_0603_1608Metric" V 2650 3000 50  0001 C CNN
 F 3 "~" V 2650 3000 50  0001 C CNN
 	1    2650 3000
@@
 F 0 "D5" H 2650 3035 50  0000 C CNN
 F 1 "LED_Small" H 2650 2944 50  0000 C CNN
-F 2 "" V 2650 2800 50  0001 C CNN
+F 2 "LED_SMD:LED_0603_1608Metric" V 2650 2800 50  0001 C CNN
 F 3 "~" V 2650 2800 50  0001 C CNN
 	1    2650 2800
@@
 F 0 "D4" H 2650 2935 50  0000 C CNN
 F 1 "LED_Small" H 2650 2844 50  0000 C CNN
-F 2 "" V 2650 2700 50  0001 C CNN
+F 2 "LED_SMD:LED_0603_1608Metric" V 2650 2700 50  0001 C CNN
 F 3 "~" V 2650 2700 50  0001 C CNN
 	1    2650 2700
@@
 F 0 "D3" H 2650 2735 50  0000 C CNN
 F 1 "LED_Small" H 2650 2644 50  0000 C CNN
-F 2 "" V 2650 2500 50  0001 C CNN
+F 2 "LED_SMD:LED_0603_1608Metric" V 2650 2500 50  0001 C CNN
 F 3 "~" V 2650 2500 50  0001 C CNN
 	1    2650 2500
@@
 F 0 "SW1" H 3500 3685 50  0000 C CNN
 F 1 "SW_Push" H 3500 3594 50  0000 C CNN
-F 2 "" H 3500 3600 50  0001 C CNN
+F 2 "Button_Switch_SMD:SW_SPST_B3U-1000P" H 3500 3600 50  0001 C CNN
 F 3 "" H 3500 3600 50  0001 C CNN
 	1    3500 3400

Commit message: More placement, more issues
Parts:
- removed D3, D4, D5, D6: LED_Small, LED_SMD:LED_0603_1608Metric, symbol Device:LED_Small
- removed R15: 360R, Resistor_SMD:R_0603_1608Metric, symbol Device:R_Small
- removed R16, R17, R18: R_Small, Resistor_SMD:R_0603_1608Metric, symbol Device:R_Small
- D2: value Green -> VDDMCU_LED
- SW1: value SW_Push -> MCU_RESET
Connections:
- net labels added: ~MCU_RESET~
- wire segments 93 -> 67
Other:
- moved on the sheet: SW1
Changed lines of the file:
@@
 $Descr A4 11693 8268
 encoding utf-8
-Sheet 4 4
+Sheet 3 4
 Title ""
 Date ""
@@
 Text Label 5600 3600 0    50   ~ 0
 VBUSDETECT
-Text HLabel 3250 2350 0    50   Input ~ 0
+Text HLabel 3250 2500 0    50   Input ~ 0
 PORT2_PWR
 Text HLabel 3250 2600 0    50   Input ~ 0
 PORT3_PWR
+Text HLabel 3250 2800 0    50   Input ~ 0
+PORT4_PWR
 Text HLabel 3250 2900 0    50   Input ~ 0
-PORT4_PWR
-Text HLabel 3250 3100 0    50   Input ~ 0
 PORT5_PWR
 Text HLabel 3350 3500 0    50   Input ~ 0
@@
 P 6000 2250
 F 0 "D2" H 6100 2300 50  0000 C CNN
-F 1 "Green" H 6000 2400 50  0000 C CNN
+F 1 "VDDMCU_LED" H 6000 2400 50  0000 C CNN
 F 2 "LED_SMD:LED_0603_1608Metric" V 6000 2250 50  0001 C CNN
 F 3 "~" V 6000 2250 50  0001 C CNN
@@
 Wire Wire Line
 	4950 2100 5400 2100
-$Comp
-L Device:R_Small R15
-U 1 1 5BD79CE0
-P 3350 2500
-F 0 "R15" V 3350 2500 50  0000 C CNN
-F 1 "360R" V 3245 2500 50  0000 C CNN
-F 2 "Resistor_SMD:R_0603_1608Metric" H 3350 2500 50  0001 C CNN
-F 3 "~" H 3350 2500 50  0001 C CNN
-	1    3350 2500
-	0    1    1    0
-$EndComp
-$Comp
-L Device:R_Small R16
-U 1 1 5BD79D36
-P 3350 2700
-F 0 "R16" V 3154 2700 50  0000 C CNN
-F 1 "R_Small" V 3245 2700 50  0000 C CNN
-F 2 "Resistor_SMD:R_0603_1608Metric" H 3350 2700 50  0001 C CNN
-F 3 "~" H 3350 2700 50  0001 C CNN
-	1    3350 2700
-	0    1    1    0
-$EndComp
-$Comp
-L Device:R_Small R17
-U 1 1 5BD79D62
-P 3350 2800
-F 0 "R17" V 3154 2800 50  0000 C CNN
-F 1 "R_Small" V 3245 2800 50  0000 C CNN
-F 2 "Resistor_SMD:R_0603_1608Metric" H 3350 2800 50  0001 C CNN
-F 3 "~" H 3350 2800 50  0001 C CNN
-	1    3350 2800
-	0    1    1    0
-$EndComp
-$Comp
-L Device:R_Small R18
-U 1 1 5BD79D90
-P 3350 3000
-F 0 "R18" V 3154 3000 50  0000 C CNN
-F 1 "R_Small" V 3245 3000 50  0000 C CNN
-F 2 "Resistor_SMD:R_0603_1608Metric" H 3350 3000 50  0001 C CNN
-F 3 "~" H 3350 3000 50  0001 C CNN
-	1    3350 3000
-	0    1    1    0
-$EndComp
-Wire Wire Line
-	3800 2500 3500 2500
-Wire Wire Line
-	3500 2500 3500 2350
-Wire Wire Line
-	3500 2350 3250 2350
-Connection ~ 3500 2500
-Wire Wire Line
-	3500 2500 3450 2500
-Wire Wire Line
-	3800 2600 3500 2600
-Wire Wire Line
-	3500 2600 3500 2700
-Wire Wire Line
-	3500 2700 3450 2700
-Wire Wire Line
-	3500 2600 3250 2600
-Connection ~ 3500 2600
-Wire Wire Line
-	3800 2800 3500 2800
-Wire Wire Line
-	3500 2800 3500 2900
-Wire Wire Line
-	3500 2900 3250 2900
-Connection ~ 3500 2800
-Wire Wire Line
-	3500 2800 3450 2800
 NoConn ~ 3800 3100
 NoConn ~ 3800 3000
-Wire Wire Line
-	3800 2900 3550 2900
-Wire Wire Line
-	3550 2900 3550 3000
-Wire Wire Line
-	3550 3100 3250 3100
-Wire Wire Line
-	3550 3000 3450 3000
-Connection ~ 3550 3000
-Wire Wire Line
-	3550 3000 3550 3100
-$Comp
-L Device:LED_Small D6
-U 1 1 5BD9534D
-P 2650 3000
-F 0 "D6" H 2650 3235 50  0000 C CNN
-F 1 "LED_Small" H 2650 3144 50  0000 C CNN
-F 2 "LED_SMD:LED_0603_1608Metric" V 2650 3000 50  0001 C CNN
-F 3 "~" V 2650 3000 50  0001 C CNN
-	1    2650 3000
-	1    0    0    -1
-$EndComp
-$Comp
-L Device:LED_Small D5
-U 1 1 5BD95397
-P 2650 2800
-F 0 "D5" H 2650 3035 50  0000 C CNN
-F 1 "LED_Small" H 2650 2944 50  0000 C CNN
-F 2 "LED_SMD:LED_0603_1608Metric" V 2650 2800 50  0001 C CNN
-F 3 "~" V 2650 2800 50  0001 C CNN
-	1    2650 2800
-	1    0    0    -1
-$EndComp
-$Comp
-L Device:LED_Small D4
-U 1 1 5BD953CF
-P 2650 2700
-F 0 "D4" H 2650 2935 50  0000 C CNN
-F 1 "LED_Small" H 2650 2844 50  0000 C CNN
-F 2 "LED_SMD:LED_0603_1608Metric" V 2650 2700 50  0001 C CNN
-F 3 "~" V 2650 2700 50  0001 C CNN
-	1    2650 2700
-	1    0    0    -1
-$EndComp
-$Comp
-L Device:LED_Small D3
-U 1 1 5BD95435
-P 2650 2500
-F 0 "D3" H 2650 2735 50  0000 C CNN
-F 1 "LED_Small" H 2650 2644 50  0000 C CNN
-F 2 "LED_SMD:LED_0603_1608Metric" V 2650 2500 50  0001 C CNN
-F 3 "~" V 2650 2500 50  0001 C CNN
-	1    2650 2500
-	1    0    0    -1
-$EndComp
-$Comp
-L power:GND #PWR060
-U 1 1 5BD954D4
-P 2100 2750
-F 0 "#PWR060" H 2100 2500 50  0001 C CNN
-F 1 "GND" H 2105 2577 50  0000 C CNN
-F 2 "" H 2100 2750 50  0001 C CNN
-F 3 "" H 2100 2750 50  0001 C CNN
-	1    2100 2750
-	1    0    0    -1
-$EndComp
-Wire Wire Line
-	2550 3000 2300 3000
-Wire Wire Line
-	2300 3000 2300 2800
-Wire Wire Line
-	2300 2700 2100 2700
-Wire Wire Line
-	2100 2700 2100 2750
-Wire Wire Line
-	2550 2700 2300 2700
-Connection ~ 2300 2700
-Wire Wire Line
-	2550 2800 2300 2800
-Connection ~ 2300 2800
-Wire Wire Line
-	2300 2800 2300 2700
-Wire Wire Line
-	2550 2500 2300 2500
-Wire Wire Line
-	2300 2500 2300 2700
-Wire Wire Line
-	3250 2500 2750 2500
-Wire Wire Line
-	2750 2700 3250 2700
-Wire Wire Line
-	3250 2800 2750 2800
-Wire Wire Line
-	2750 3000 3250 3000
 NoConn ~ 5450 3700
 NoConn ~ 5450 2900
@@
 L Switch:SW_Push SW1
 U 1 1 5BDBABA3
-P 3500 3400
-F 0 "SW1" H 3500 3685 50  0000 C CNN
-F 1 "SW_Push" H 3500 3594 50  0000 C CNN
-F 2 "Button_Switch_SMD:SW_SPST_B3U-1000P" H 3500 3600 50  0001 C CNN
-F 3 "" H 3500 3600 50  0001 C CNN
-	1    3500 3400
+P 3150 3400
+F 0 "SW1" H 3150 3685 50  0000 C CNN
+F 1 "MCU_RESET" H 3150 3594 50  0000 C CNN
+F 2 "Button_Switch_SMD:SW_SPST_B3U-1000P" H 3150 3600 50  0001 C CNN
+F 3 "" H 3150 3600 50  0001 C CNN
+	1    3150 3400
 	1    0    0    -1
 $EndComp
@@
 L power:GND #PWR0101
 U 1 1 5BDBAC4F
-P 3200 3400
-F 0 "#PWR0101" H 3200 3150 50  0001 C CNN
-F 1 "GND" V 3205 3272 50  0000 R CNN
-F 2 "" H 3200 3400 50  0001 C CNN
-F 3 "" H 3200 3400 50  0001 C CNN
-	1    3200 3400
+P 2800 3400
+F 0 "#PWR0101" H 2800 3150 50  0001 C CNN
+F 1 "GND" V 2805 3272 50  0000 R CNN
+F 2 "" H 2800 3400 50  0001 C CNN
+F 3 "" H 2800 3400 50  0001 C CNN
+	1    2800 3400
 	0    1    1    0
 $EndComp
 Wire Wire Line
-	3300 3400 3200 3400
-Wire Wire Line
-	3700 3400 3800 3400
+	3350 3400 3800 3400
 $Comp
 L Power_Extra:VDDMCU #PWR0106
@@
 Wire Wire Line
 	5500 1800 5500 1750
+Wire Wire Line
+	3250 2600 3800 2600
+Wire Wire Line
+	3250 2500 3800 2500
+Wire Wire Line
+	3250 2800 3800 2800
+Wire Wire Line
+	3250 2900 3800 2900
+Text Label 3750 3400 2    50   ~ 0
+~MCU_RESET~
+Wire Wire Line
+	2950 3400 2800 3400
 $EndSCHEMATC

Commit message: More routing, simplification
Parts:
- added J10: DBG_UART, Connector_JST:JST_SH_BM04B-SRSS-TB_1x04-1MP_P1.00mm_Vertical, symbol Connector_Generic:Conn_01x04
Connections:
- wire segments 67 -> 73
- no-connect marks 12 -> 10
Changed lines of the file:
@@
 Text Label 5600 3600 0    50   ~ 0
 VBUSDETECT
-Text HLabel 3250 2500 0    50   Input ~ 0
+Text HLabel 5995 2800 2    50   Input ~ 0
 PORT2_PWR
-Text HLabel 3250 2600 0    50   Input ~ 0
+Text HLabel 5995 2700 2    50   Input ~ 0
 PORT3_PWR
-Text HLabel 3250 2800 0    50   Input ~ 0
+Text HLabel 5995 2600 2    50   Input ~ 0
 PORT4_PWR
-Text HLabel 3250 2900 0    50   Input ~ 0
+Text HLabel 6000 2500 2    50   Input ~ 0
 PORT5_PWR
 Text HLabel 3350 3500 0    50   Input ~ 0
@@
 Text HLabel 3350 3600 0    50   Input ~ 0
 PORT3_EN
-Text HLabel 3350 3700 0    50   Input ~ 0
+Text HLabel 3350 3800 0    50   Input ~ 0
 PORT4_EN
-Text HLabel 3350 3800 0    50   Input ~ 0
+Text HLabel 5900 3700 2    50   Input ~ 0
 PORT5_EN
 Wire Wire Line
@@
 	3350 3600 3800 3600
 Wire Wire Line
-	3800 3700 3350 3700
-Wire Wire Line
-	3800 3800 3350 3800
+	5450 3700 5900 3700
 $Comp
 L Device:C_Small C15
@@
 NoConn ~ 3800 3100
 NoConn ~ 3800 3000
-NoConn ~ 5450 3700
-NoConn ~ 5450 2900
-NoConn ~ 5450 2800
-NoConn ~ 5450 2700
-NoConn ~ 5450 2600
-NoConn ~ 5450 2500
 NoConn ~ 3800 2700
 Wire Wire Line
@@
 Wire Wire Line
 	5500 1800 5500 1750
-Wire Wire Line
-	3250 2600 3800 2600
-Wire Wire Line
-	3250 2500 3800 2500
-Wire Wire Line
-	3250 2800 3800 2800
-Wire Wire Line
-	3250 2900 3800 2900
 Text Label 3750 3400 2    50   ~ 0
 ~MCU_RESET~
 Wire Wire Line
 	2950 3400 2800 3400
+Wire Wire Line
+	3800 3800 3350 3800
+NoConn ~ 3800 3700
+Wire Wire Line
+	6000 2500 5450 2500
+Wire Wire Line
+	6000 2600 5450 2600
+Wire Wire Line
+	6000 2700 5450 2700
+Wire Wire Line
+	6000 2800 5450 2800
+NoConn ~ 5450 2900
+NoConn ~ 3800 2900
+NoConn ~ 3800 2800
+$Comp
+L Connector_Generic:Conn_01x04 J10
+U 1 1 5C07D882
+P 3100 2600
+F 0 "J10" H 3100 2300 50  0000 C CNN
+F 1 "DBG_UART" V 3200 2550 50  0000 C CNN
+F 2 "Connector_JST:JST_SH_BM04B-SRSS-TB_1x04-1MP_P1.00mm_Vertical" H 3100 2600 50  0001 C CNN
+F 3 "~" H 3100 2600 50  0001 C CNN
+	1    3100 2600
+	-1   0    0    1
+$EndComp
+Wire Wire Line
+	3800 2500 3300 2500
+Wire Wire Line
+	3800 2600 3300 2600
+$Comp
+L power:GND #PWR066
+U 1 1 5C080544
+P 3350 2750
+F 0 "#PWR066" H 3350 2500 50  0001 C CNN
+F 1 "GND" H 3355 2577 50  0000 C CNN
+F 2 "" H 3350 2750 50  0001 C CNN
+F 3 "" H 3350 2750 50  0001 C CNN
+	1    3350 2750
+	1    0    0    -1
+$EndComp
+Wire Wire Line
+	3300 2700 3350 2700
+Wire Wire Line
+	3350 2700 3350 2750
+$Comp
+L Power_Extra:VDDMCU #PWR061
+U 1 1 5C081E76
+P 3350 2300
+F 0 "#PWR061" H 3350 2150 50  0001 C CNN
+F 1 "VDDMCU" H 3365 2473 50  0000 C CNN
+F 2 "" H 3350 2300 50  0001 C CNN
+F 3 "" H 3350 2300 50  0001 C CNN
+	1    3350 2300
+	1    0    0    -1
+$EndComp
+Wire Wire Line
+	3300 2400 3350 2400
+Wire Wire Line
+	3350 2400 3350 2300
 $EndSCHEMATC
